Commit message: diff_drive controller and joint state broadcaster

File: fusion_rover/urdf/fusionrover.urdf.xacro (robot description, xacro)
@@ -1,35 +1,33 @@
 <?xml version="1.0"?>
 <robot name="fusionrover" xmlns:xacro="http://www.ros.org/wiki/xacro">
+  <material name="gray"><color rgba="0.5 0.5 0.5 1.0"/></material>
+  <material name="black"><color rgba="0.0 0.0 0.0 1.0"/></material>
   <xacro:property name="chassis_mass"   value="10.0"/>
   <xacro:property name="chassis_length" value="0.45"/>
   <xacro:property name="chassis_width"  value="0.30"/>
   <xacro:property name="chassis_height" value="0.12"/>
-  <xacro:property name="wheel_mass"   value="1.0"/>
-  <xacro:property name="wheel_radius" value="0.06"/>
-  <xacro:property name="wheel_width"  value="0.04"/>
+  <xacro:property name="wheel_mass"     value="1.0"/>
+  <xacro:property name="wheel_radius"   value="0.06"/>
+  <xacro:property name="wheel_width"    value="0.04"/>
   <xacro:property name="wheel_x_offset" value="0.18"/>
   <xacro:property name="wheel_y_offset" value="0.16"/>
   <xacro:property name="ground_clearance" value="0.02"/>
-  <material name="gray">
-    <color rgba="0.5 0.5 0.5 1.0"/>
-  </material>
-  <material name="black">
-    <color rgba="0.0 0.0 0.0 1.0"/>
-  </material>
+  <link name="base_footprint"/>
+  <joint name="base_footprint_joint" type="fixed">
+    <parent link="base_footprint"/>
+    <child link="base_link"/>
+    <origin xyz="0 0 ${chassis_height/2 + ground_clearance}" rpy="0 0 0"/>
+  </joint>
   <link name="base_link">
     <visual>
-      <geometry>
-        <box size="${chassis_length} ${chassis_width} ${chassis_height}"/>
-      </geometry>
+      <geometry><box size="${chassis_length} ${chassis_width} ${chassis_height}"/></geometry>
       <material name="gray"/>
     </visual>
     <collision>
-      <geometry>
-        <box size="${chassis_length} ${chassis_width} ${chassis_height}"/>
-      </geometry>
+      <geometry><box size="${chassis_length} ${chassis_width} ${chassis_height}"/></geometry>
     </collision>
     <inertial>
       <mass value="${chassis_mass}"/>
-      <origin xyz="0 0 0"/>
+      <origin xyz="0 0 0" rpy="0 0 0"/>
       <inertia
         ixx="${(1/12) * chassis_mass * (chassis_width*chassis_width + chassis_height*chassis_height)}"
@@ -40,24 +38,18 @@
     </inertial>
   </link>
-  <gazebo reference="base_link">
-    <material>Gazebo/Grey</material>
-  </gazebo>
   <xacro:macro name="wheel" params="name x y">
     <link name="${name}">
       <visual>
-        <geometry>
-          <cylinder radius="${wheel_radius}" length="${wheel_width}"/>
-        </geometry>
-        <origin xyz="0 0 0" rpy="1.5708 0 0"/>
+        <origin rpy="${pi/2} 0 0" xyz="0 0 0"/>
+        <geometry><cylinder radius="${wheel_radius}" length="${wheel_width}"/></geometry>
         <material name="black"/>
       </visual>
       <collision>
-        <geometry>
-          <cylinder radius="${wheel_radius}" length="${wheel_width}"/>
-        </geometry>
-        <origin xyz="0 0 0" rpy="1.5708 0 0"/>
+        <origin rpy="${pi/2} 0 0" xyz="0 0 0"/>
+        <geometry><cylinder radius="${wheel_radius}" length="${wheel_width}"/></geometry>
       </collision>
       <inertial>
         <mass value="${wheel_mass}"/>
+        <origin rpy="${pi/2} 0 0" xyz="0 0 0"/>
         <inertia
           ixx="${(1/12)*wheel_mass*(3*wheel_radius*wheel_radius + wheel_width*wheel_width)}"
@@ -76,6 +68,6 @@
     <gazebo reference="${name}">
       <material>Gazebo/Black</material>
-      <mu1 value="1.0"/>
-      <mu2 value="1.0"/>
+      <mu1>1.0</mu1>
+      <mu2>1.0</mu2>
     </gazebo>
   </xacro:macro>
@@ -84,3 +76,29 @@
   <xacro:wheel name="rear_left_wheel"   x="-${wheel_x_offset}" y="${wheel_y_offset}"/>
   <xacro:wheel name="rear_right_wheel"  x="-${wheel_x_offset}" y="-${wheel_y_offset}"/>
+  <ros2_control name="FusionRoverSystem" type="system">
+    <hardware>
+      <plugin>gazebo_ros2_control/GazeboSystem</plugin>
+    </hardware>
+    <joint name="front_left_wheel_joint">
+      <command_interface name="velocity"/>
+      <state_interface name="position"/><state_interface name="velocity"/>
+    </joint>
+    <joint name="front_right_wheel_joint">
+      <command_interface name="velocity"/>
+      <state_interface name="position"/><state_interface name="velocity"/>
+    </joint>
+    <joint name="rear_left_wheel_joint">
+      <command_interface name="velocity"/>
+      <state_interface name="position"/><state_interface name="velocity"/>
+    </joint>
+    <joint name="rear_right_wheel_joint">
+      <command_interface name="velocity"/>
+      <state_interface name="position"/><state_interface name="velocity"/>
+    </joint>
+  </ros2_control>
+  <gazebo>
+    <plugin name="gazebo_ros2_control" filename="libgazebo_ros2_control.so">
+      <parameters>$(find fusion_rover)/config/diff_drive_controller.yaml</parameters>
+    </plugin>
+  </gazebo>
 </robot>

Commit message: lidar and ultrasonic senor

File: fusion_rover/urdf/fusionrover.urdf.xacro (robot description, xacro)
@@ -38,4 +38,54 @@
     </inertial>
   </link>
+  <link name="lidar_link">
+    <visual>
+      <geometry>
+        <cylinder radius="0.03" length="0.02"/>
+      </geometry>
+      <material name="black"/>
+    </visual>
+    <collision>
+      <geometry>
+        <cylinder radius="0.03" length="0.02"/>
+      </geometry>
+    </collision>
+    <inertial>
+      <mass value="0.1"/>
+      <origin xyz="0 0 0" rpy="0 0 0"/>
+      <inertia ixx="0.0001" ixy="0.0" ixz="0.0"
+               iyy="0.0001" iyz="0.0"
+               izz="0.0001"/>
+    </inertial>
+  </link>
+  <joint name="lidar_joint" type="fixed">
+    <parent link="base_link"/>
+    <child link="lidar_link"/>
+    <origin xyz="0.18 0 0.10" rpy="0 0 0"/>
+  </joint>
+  <link name="ultrasonic_front_link">
+    <visual>
+      <geometry>
+        <box size="0.04 0.02 0.02"/>
+      </geometry>
+      <material name="black"/>
+    </visual>
+    <collision>
+      <geometry>
+        <box size="0.04 0.02 0.02"/>
+      </geometry>
+    </collision>
+    <inertial>
+      <mass value="0.05"/>
+      <origin xyz="0 0 0" rpy="0 0 0"/>
+      <inertia ixx="0.00005" ixy="0.0" ixz="0.0"
+               iyy="0.00005" iyz="0.0"
+               izz="0.00005"/>
+    </inertial>
+  </link>
+  <joint name="ultrasonic_front_joint" type="fixed">
+    <parent link="base_link"/>
+    <child link="ultrasonic_front_link"/>
+    <origin xyz="0.23 0 0.06" rpy="0 0 0"/>
+  </joint>
   <xacro:macro name="wheel" params="name x y">
     <link name="${name}">
@@ -103,3 +153,77 @@
     </plugin>
   </gazebo>
+  <gazebo reference="lidar_link">
+    <sensor name="lidar_sensor" type="ray">
+      <pose>0 0 0 0 0 0</pose>
+      <update_rate>10</update_rate>
+      <visualize>true</visualize>
+      <ray>
+        <scan>
+          <horizontal>
+            <samples>360</samples>
+            <resolution>1</resolution>
+            <min_angle>-3.14159</min_angle>
+            <max_angle>3.14159</max_angle>
+          </horizontal>
+        </scan>
+        <range>
+          <min>0.12</min>
+          <max>10.0</max>
+          <resolution>0.01</resolution>
+        </range>
+        <noise>
+          <type>gaussian</type>
+          <mean>0.0</mean>
+          <stddev>0.01</stddev>
+        </noise>
+      </ray>
+      <plugin name="gazebo_ros_laser" filename="libgazebo_ros_ray_sensor.so">
+        <ros>
+          <remapping>~/out:=scan</remapping>
+        </ros>
+        <output_type>sensor_msgs/LaserScan</output_type>
+        <frame_name>lidar_link</frame_name>
+      </plugin>
+    </sensor>
+  </gazebo>
+  <gazebo reference="ultrasonic_front_link">
+    <sensor name="ultrasonic_front_sensor" type="ray">
+      <pose>0 0 0 0 0 0</pose>
+      <update_rate>20</update_rate>
+      <visualize>true</visualize>
+      <ray>
+        <scan>
+          <horizontal>
+            <samples>5</samples> <resolution>1</resolution>
+            <min_angle>-0.1</min_angle>
+            <max_angle>0.1</max_angle>
+          </horizontal>
+          <vertical>
+             <samples>5</samples>
+             <resolution>1</resolution>
+             <min_angle>-0.1</min_angle>
+             <max_angle>0.1</max_angle>
+          </vertical>
+        </scan>
+        <range>
+          <min>0.02</min>
+          <max>4.0</max>
+          <resolution>0.01</resolution>
+        </range>
+        <noise>
+          <type>gaussian</type>
+          <mean>0.0</mean>
+          <stddev>0.005</stddev>
+        </noise>
+      </ray>
+      <plugin name="gazebo_ros_range" filename="libgazebo_ros_ray_sensor.so">
+        <ros>
+          <remapping>~/out:=ultrasonic/front</remapping>
+        </ros>
+        <output_type>sensor_msgs/Range</output_type>
+        <frame_name>ultrasonic_front_link</frame_name>
+        <radiation_type>ultrasound</radiation_type>
+      </plugin>
+    </sensor>
+  </gazebo>
 </robot>
